File: sensor-project/sensor-project.kicad_sch (KiCad schematic)
At the start: 22 parts, among them J1 Conn_01x08, J2 Conn_01x08, J3 Conn_01x08, U1 picoscope-2000, U2 74HC4051, U3 74HC4051, U4 74HC4051, U5 4094

Commit message: sdfsdfds
Parts:
- U4: RSpart 103-8177 -> (none)
Connections:
- net GND: no longer J1.1 (Pin_1), J2.1 (Pin_1), U2.13 (A0), U3.13 (A0)
- net at J3.1 (Pin_1), U4.13 (A0): now also J2.1 (Pin_1), U3.13 (A0); no longer J2.2 (Pin_2), U3.14 (A1)
- new net: J1.1 (Pin_1), U2.13 (A0)
- new net: J2.2 (Pin_2), U3.14 (A1)
Changed lines of the file:
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@@
 (kicad_sch (version 20230121) (generator eeschema)
   (paper "A4")
-  (junction (at 181.61 28.575) (diameter 0) (color 0 0 0 0)
-  )
   (junction (at 187.325 69.215) (diameter 0) (color 0 0 0 0)
   )
   (junction (at 78.74 186.69) (diameter 0) (color 0 0 0 0)
   )
-  (junction (at 184.785 31.115) (diameter 0) (color 0 0 0 0)
-  )
   (junction (at 254 79.375) (diameter 0) (color 0 0 0 0)
   )
@@
   (junction (at 217.17 81.915) (diameter 0) (color 0 0 0 0)
   )
+  (junction (at 184.785 28.575) (diameter 0) (color 0 0 0 0)
+  )
   (junction (at 231.14 127.635) (diameter 0) (color 0 0 0 0)
   )
@@
   (junction (at 207.645 90.805) (diameter 0) (color 0 0 0 0)
   )
-  (junction (at 180.975 66.675) (diameter 0) (color 0 0 0 0)
-  )
   (wire (pts (xy 66.04 177.8) (xy 45.72 177.8))
     (stroke (width 0) (type default))
@@
     (stroke (width 0) (type default))
   )
-  (wire (pts (xy 184.785 31.115) (xy 212.09 31.115))
+  (wire (pts (xy 173.99 31.115) (xy 212.09 31.115))
     (stroke (width 0) (type default))
   )
@@
     (stroke (width 0) (type default))
   )
-  (wire (pts (xy 181.61 28.575) (xy 212.09 28.575))
-    (stroke (width 0) (type default))
-  )
-  (wire (pts (xy 173.99 31.115) (xy 184.785 31.115))
+  (wire (pts (xy 173.99 28.575) (xy 184.785 28.575))
     (stroke (width 0) (type default))
   )
@@
     (stroke (width 0) (type default))
   )
-  (wire (pts (xy 175.895 66.675) (xy 180.975 66.675))
-    (stroke (width 0) (type default))
-  )
   (wire (pts (xy 175.26 116.205) (xy 220.98 116.205))
     (stroke (width 0) (type default))
@@
     (stroke (width 0) (type default))
   )
-  (wire (pts (xy 184.785 31.115) (xy 184.785 103.505))
-    (stroke (width 0) (type default))
-  )
   (wire (pts (xy 238.76 111.125) (xy 246.38 111.125))
     (stroke (width 0) (type default))
@@
     (stroke (width 0) (type default))
   )
+  (wire (pts (xy 184.785 28.575) (xy 184.785 103.505))
+    (stroke (width 0) (type default))
+  )
   (wire (pts (xy 173.99 33.655) (xy 212.09 33.655))
     (stroke (width 0) (type default))
@@
     (stroke (width 0) (type default))
   )
-  (wire (pts (xy 180.975 66.675) (xy 197.485 66.675))
+  (wire (pts (xy 175.895 66.675) (xy 197.485 66.675))
     (stroke (width 0) (type default))
   )
@@
     (stroke (width 0) (type default))
   )
-  (wire (pts (xy 180.975 61.595) (xy 180.975 66.675))
-    (stroke (width 0) (type default))
-  )
   (wire (pts (xy 114.935 170.18) (xy 99.695 170.18))
     (stroke (width 0) (type default))
@@
     (stroke (width 0) (type default))
   )
-  (wire (pts (xy 173.99 28.575) (xy 181.61 28.575))
-    (stroke (width 0) (type default))
-  )
   (wire (pts (xy 222.25 52.705) (xy 231.775 52.705))
     (stroke (width 0) (type default))
@@
     (stroke (width 0) (type default))
   )
-  (wire (pts (xy 181.61 23.495) (xy 181.61 28.575))
-    (stroke (width 0) (type default))
-  )
   (wire (pts (xy 102.235 175.26) (xy 91.44 175.26))
     (stroke (width 0) (type default))
@@
   )
   (wire (pts (xy 40.005 180.34) (xy 57.15 180.34))
+    (stroke (width 0) (type default))
+  )
+  (wire (pts (xy 184.785 28.575) (xy 212.09 28.575))
     (stroke (width 0) (type default))
   )
@@
       (effects (font (size 1.27 1.27)) hide)
     )
-    (property "RSpart" "103-8177" (at 231.14 111.125 0)
+    (property "RSpart" "" (at 231.14 111.125 0)
       (effects (font (size 1.27 1.27)) hide)
     )
@@
     )
   )
-  (symbol (lib_id "power:GND") (at 180.975 61.595 180) (unit 1)
-    (in_bom yes) (on_board yes) (dnp no)
-    (property "Reference" "#PWR011" (at 180.975 55.245 0)
-      (effects (font (size 1.27 1.27)) hide)
-    )
-    (property "Value" "GND" (at 177.8 59.69 0)
-      (effects (font (size 1.27 1.27)))
-    )
-    (property "Footprint" "" (at 180.975 61.595 0)
-      (effects (font (size 1.27 1.27)) hide)
-    )
-    (property "Datasheet" "" (at 180.975 61.595 0)
-      (effects (font (size 1.27 1.27)) hide)
-    )
-    (pin "1")
-    (instances
-      (project "sensor-project"
-        (path "/626b35b1-867d-4ca7-a50d-226e2d5d6721"
-          (reference "#PWR011") (unit 1)
-        )
-      )
-    )
-  )
   (symbol (lib_id "000_Resistors_Immo:100r") (at 217.17 85.725 90) (unit 1)
     (in_bom yes) (on_board yes) (dnp no) (fields_autoplaced)
@@
         (path "/626b35b1-867d-4ca7-a50d-226e2d5d6721"
           (reference "R4") (unit 1)
-        )
-      )
-    )
-  )
-  (symbol (lib_id "power:GND") (at 181.61 23.495 180) (unit 1)
-    (in_bom yes) (on_board yes) (dnp no)
-    (property "Reference" "#PWR010" (at 181.61 17.145 0)
-      (effects (font (size 1.27 1.27)) hide)
-    )
-    (property "Value" "GND" (at 178.435 21.59 0)
-      (effects (font (size 1.27 1.27)))
-    )
-    (property "Footprint" "" (at 181.61 23.495 0)
-      (effects (font (size 1.27 1.27)) hide)
-    )
-    (property "Datasheet" "" (at 181.61 23.495 0)
-      (effects (font (size 1.27 1.27)) hide)
-    )
-    (pin "1")
-    (instances
-      (project "sensor-project"
-        (path "/626b35b1-867d-4ca7-a50d-226e2d5d6721"
-          (reference "#PWR010") (unit 1)
         )
       )
@@
     (pin "2")
     (pin "3")
+    (pin "4")
     (pin "5")
-    (pin "4")
     (pin "6")
     (instances
